File: PCB/Badge_Bottom/Badge_Bottom.kicad_sch (KiCad schematic)
At the start: 27 parts, among them J1 Nylon Screw, J10 Debug, J18 Debug, J2 Metal Screw, J3 Nylon Screw, J4 Metal Screw, J5 Nylon Screw, J6 Metal Screw, Q1 AO3400A, U2 CH32V305RBT6, Y1 8M

Commit message: finised pcb layout
Parts:
- removed Q1: AO3400A, Package_TO_SOT_SMD:SOT-23, symbol Transistor_FET:AO3400A
- added C13 (x2): 10u, Capacitor_Tantalum_SMD:CP_EIA-3216-18_Kemet-A, symbol Device:C_Polarized_Small
- added C2, C3: 1u, Capacitor_SMD:C_0603_1608Metric, symbol Device:C_Small
- added C3 (x2): 2u2, Capacitor_SMD:C_0603_1608Metric, symbol Device:C_Small
- added C3 (x2): 2n2, Capacitor_SMD:C_0603_1608Metric, symbol Device:C_Small
- added C3 (x2): 0.1u, Capacitor_SMD:C_0603_1608Metric, symbol Device:C_Small
- added JP1 (x3): SolderJumper_3_Bridged12, Jumper:SolderJumper-3_P1.3mm_Bridged12_RoundedPad1.0x1.5mm, symbol Jumper:SolderJumper_3_Bridged12
- added JP5: SolderJumper_2_Bridged, Jumper:SolderJumper-2_P1.3mm_Bridged_RoundedPad1.0x1.5mm, symbol Jumper:SolderJumper_2_Bridged
- added Q1: AO3401A, Package_TO_SOT_SMD:SOT-23, symbol Transistor_FET:AO3401A
- added Q2: AO3400A, Package_TO_SOT_SMD:SOT-23, symbol Transistor_FET:AO3400A
- added R3 (x2): 470, Resistor_SMD:R_0603_1608Metric, symbol Device:R_Small
- added R3 (x3): 22, Resistor_SMD:R_0603_1608Metric, symbol Device:R_Small
- added R3: 10k, Resistor_SMD:R_0603_1608Metric, symbol Device:R_Small
- added TP1 (x11): TestPoint, TestPoint:TestPoint_Pad_D1.0mm, symbol Connector:TestPoint
- added U3: PCM5100A, Package_SO:TSSOP-20_4.4x6.5mm_P0.65mm, symbol Audio:PCM5100A
- added U4: XC6206PxxxMR, Package_TO_SOT_SMD:SOT-23-3, symbol Regulator_Linear:XC6206PxxxMR
- J18: footprint Connector_PinSocket_2.54mm:PinSocket_2x02_P2.54mm_Horizontal -> 2x02_pinsocket_254:HDR-TH_4P-P2.54-H-F-R2-C2-W8.5
Connections:
- net PB14-BTNL_UP is gone; now on net PB12-BNTR_DOWN: U2.35 (PB14)
- net +3V3: now also JP1.1 (A), JP1.3 (B), JP1.3 (B), U3.20 (DVDD); no longer R3.1
- net BOOT0: now also TP1.1
- net GND: now also J1.1 (Pin_1), C13.2, C2.1, C3.1, C3.2, JP1.1 (A), JP1.1 (A), JP1.3 (B), JP5.1 (A), Q2.2 (S), R3.2, U3.16 (FMT), U3.19 (DGND), U4.1 (GND)
- net NRST: now also TP1.1
- net PA1-ADC_IN1: now also TP1.1
- net PA6-LEDFET: now also Q2.1 (G), R3.1; no longer R3.2
- net PA8-TIM1: now also TP1.1
- net PB12-BNTR_DOWN: no longer U2.33 (PB12)
- net VDD: now also R3.2, C3.2, Q1.2 (S), U4.3 (VI); no longer J5.1 (Pin_1)
- net at R3.1, U2.28 (BOOT1/PB2): now also TP1.1
- net at U2.23 (PA7): now also D1.1 (K); no longer D1.2 (A)
- net at R3.1: now also D1.2 (A); no longer D1.1 (K)
- net PA0-GPIO renamed PA0-BTNL-BTN
- net PB13-BTNL-BTN renamed PB13-I2S2_CK
- net PB13-I2S2_CK: now also R3.1
- net PB15-BTNL_DOWN renamed PB15-I2S2_SD
- net PB15-I2S2_SD: now also R3.1
- net PC14-GPIO renamed PC14-BTNL_UP
- net PC15-GPIO renamed PC15-BTNL_DOWN
- new net: C3.2, U3.5 (VNEG)
- new net: R3.1, U3.6 (OUTL)
- new net: R3.2, TP1.1, U3.14 (DIN)
- new net: R3.2, TP1.1, U3.13 (BCK)
- new net: JP1.2 (C), U3.11 (FLT)
- new net: Q1.1 (G), Q2.3 (D), R3.1, TP1.1
- new net: J5.1 (Pin_1), Q1.3 (D)
- new net: R3.1, U3.7 (OUTR)
- new net: R3.2, TP1.1, U3.15 (LRCK)
- new net: JP1.2 (C), U3.17 (XSMT)
- new net: C3.1, U3.4 (CAPM)
- new net: C3.2, U3.2 (CAPP)
- new net: C13.1, C3.1, U3.18 (LDOO)
- new net: JP1.2 (C), U3.10 (DEMP)
- new net: JP5.2 (B), U3.12 (SCK)
- new net +3.3VA: C13.1, C2.2, C3.1, TP1.1, U3.1 (CPVDD), U3.8 (AVDD), U4.2 (VO)
- new net DAC_OUT_L: C3.2, R3.2
- new net DAC_OUT_R: C3.2, R3.2
- new net GNDA: C13.2, C3.1, C3.1, C3.1, C3.2, TP1.1, U3.3 (CPGND), U3.9 (AGND)
- new net PB12-I2S2_WS: R3.1, U2.33 (PB12)
Other:
- added sheet BadeLink (badgelink.kicad_sch)
- note added: "14x SK6809, running on Battery Voltage (roughly down to ~3.5V)"
- note added: "ADC Battery Measurment"
- note added: "Debug Pins, either Tag-Connect or 2,54mm Header"
- note added: "Ext. Clock, needed for 480Mhz USB Speed (might be overkill)"
- note added: "PCM5100 DAC"
- note added: "Top Badge PCB Interface"
- note added: "WCH CH32V305"
- note removed: "TODO: - Finish schematic (gpio routing) - Add proper micro SD slot (tf push) - add 2x2 pinsocket - add jstph clone for battery con - make schematic prettier"
- moved on the sheet: C3, D1, J1, J10, J18, J2, J3, J4, J5, J6, R3, U2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

Commit message: Added docs and readme, ordered PCBs at JLC
Other:
- company: (none) -> Unterland
- title: (none) -> Unterland Badge Bottom
