File: PCB/Badge_Bottom/badgelink.kicad_sch (KiCad schematic)
At the start: 34 parts, among them CN1 JACK_OUT, CN2 JACK_IN, SW4 JACK_IN_SW, SW5 JACK_IN_SW

Commit message: Added docs and readme, ordered PCBs at JLC
Other:
- company: (none) -> Unterland
- title: (none) -> Unterland Badge Bottom
Changed lines of the file:
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@@
 (kicad_sch (version 20230121) (generator eeschema)
   (paper "A4")
+  (title_block
+    (title "Unterland Badge Bottom")
+    (date "2023-07-29")
+    (rev "1")
+    (company "Unterland")
+    (comment 1 "BadgeLink Expansion Section")
+  )
   (junction (at 119.38 129.54) (diameter 0) (color 0 0 0 0)
   )
